Commit message: Xacro: added standoff rods to the robot base

File: xacro/barista_robot_model.urdf.xacro (robot description, xacro)
@@ -3,4 +3,5 @@
     <!-- Include -->
     <xacro:include filename="$(find barista_robot_description)/xacro/rviz_materials.xacro"/>
+    <xacro:include filename="$(find barista_robot_description)/xacro/standoff_rods.xacro"/>
     <!-- Properties -->
     <xacro:property name="base_plate_mass" value="0.8"/>
@@ -38,3 +39,29 @@
         <child link="base_plate_link"/>
     </joint>
+    <!-- Standoff Rods -->
+    <xacro:standoff_rods name="standoff_rods1_link" color="White"/>
+    <xacro:standoff_rods name="standoff_rods2_link" color="White"/>
+    <xacro:standoff_rods name="standoff_rods3_link" color="White"/>
+    <xacro:standoff_rods name="standoff_rods4_link" color="White"/>
+    <!-- Standoff Rods Joints-->
+    <joint name="standoff_rods1_joint" type="fixed">
+        <origin rpy="0 0 0" xyz="0.03 0.13 0.1875"/>
+        <parent link="base_plate_link"/>
+        <child link="standoff_rods1_link"/>
+    </joint>
+    <joint name="standoff_rods2_joint" type="fixed">
+        <origin rpy="0 0 0" xyz="-0.03 0.13 0.1875"/>
+        <parent link="base_plate_link"/>
+        <child link="standoff_rods2_link"/>
+    </joint>
+    <joint name="standoff_rods3_joint" type="fixed">
+        <origin rpy="0 0 0" xyz="-0.03 -0.13 0.1875"/>
+        <parent link="base_plate_link"/>
+        <child link="standoff_rods3_link"/>
+    </joint>
+    <joint name="standoff_rods4_joint" type="fixed">
+        <origin rpy="0 0 0" xyz="0.03 -0.13 0.1875"/>
+        <parent link="base_plate_link"/>
+        <child link="standoff_rods4_link"/>
+    </joint>
 </robot>

Commit message: Xacro: added standoff rods to the robot base

File: xacro/barista_robot_model.urdf.xacro (robot description, xacro)
@@ -3,4 +3,5 @@
     <!-- Include -->
     <xacro:include filename="$(find barista_robot_description)/xacro/rviz_materials.xacro"/>
+    <xacro:include filename="$(find barista_robot_description)/xacro/standoff_rods.xacro"/>
     <!-- Properties -->
     <xacro:property name="base_plate_mass" value="2.5"/>
@@ -38,3 +39,29 @@
         <child link="base_plate_link"/>
     </joint>
+    <!-- Standoff Rods -->
+    <xacro:standoff_rods name="standoff_rods1_link" color="White"/>
+    <xacro:standoff_rods name="standoff_rods2_link" color="White"/>
+    <xacro:standoff_rods name="standoff_rods3_link" color="White"/>
+    <xacro:standoff_rods name="standoff_rods4_link" color="White"/>
+    <!-- Standoff Rods Joints-->
+    <joint name="standoff_rods1_joint" type="fixed">
+        <origin rpy="0 0 0" xyz="0.03 0.13 0.1875"/>
+        <parent link="base_plate_link"/>
+        <child link="standoff_rods1_link"/>
+    </joint>
+    <joint name="standoff_rods2_joint" type="fixed">
+        <origin rpy="0 0 0" xyz="-0.03 0.13 0.1875"/>
+        <parent link="base_plate_link"/>
+        <child link="standoff_rods2_link"/>
+    </joint>
+    <joint name="standoff_rods3_joint" type="fixed">
+        <origin rpy="0 0 0" xyz="-0.03 -0.13 0.1875"/>
+        <parent link="base_plate_link"/>
+        <child link="standoff_rods3_link"/>
+    </joint>
+    <joint name="standoff_rods4_joint" type="fixed">
+        <origin rpy="0 0 0" xyz="0.03 -0.13 0.1875"/>
+        <parent link="base_plate_link"/>
+        <child link="standoff_rods4_link"/>
+    </joint>
 </robot>

File: xacro/rviz_materials.xacro (robot description, xacro)
@@ -4,3 +4,6 @@
       <color rgba="0.0 0.0 1.0 1"/>
   </material>
+  <material name="White">
+      <color rgba="1 1 1 1"/>
+  </material>
 </robot>

Commit message: Xacro: added standoff rods to the robot base

File: xacro/barista_robot_model.urdf.xacro (robot description, xacro)
@@ -3,4 +3,5 @@
     <!-- Include -->
     <xacro:include filename="$(find barista_robot_description)/xacro/rviz_materials.xacro"/>
+    <xacro:include filename="$(find barista_robot_description)/xacro/standoff_rods.xacro"/>
     <!-- Properties -->
     <xacro:property name="base_plate_mass" value="0.8"/>
@@ -38,3 +39,29 @@
         <child link="base_plate_link"/>
     </joint>
+    <!-- Standoff Rods -->
+    <xacro:standoff_rods name="standoff_rods1_link" color="White"/>
+    <xacro:standoff_rods name="standoff_rods2_link" color="White"/>
+    <xacro:standoff_rods name="standoff_rods3_link" color="White"/>
+    <xacro:standoff_rods name="standoff_rods4_link" color="White"/>
+    <!-- Standoff Rods Joints-->
+    <joint name="standoff_rods1_joint" type="fixed">
+        <origin rpy="0 0 0" xyz="0.03 0.13 0.1875"/>
+        <parent link="base_plate_link"/>
+        <child link="standoff_rods1_link"/>
+    </joint>
+    <joint name="standoff_rods2_joint" type="fixed">
+        <origin rpy="0 0 0" xyz="-0.03 0.13 0.1875"/>
+        <parent link="base_plate_link"/>
+        <child link="standoff_rods2_link"/>
+    </joint>
+    <joint name="standoff_rods3_joint" type="fixed">
+        <origin rpy="0 0 0" xyz="-0.03 -0.13 0.1875"/>
+        <parent link="base_plate_link"/>
+        <child link="standoff_rods3_link"/>
+    </joint>
+    <joint name="standoff_rods4_joint" type="fixed">
+        <origin rpy="0 0 0" xyz="0.03 -0.13 0.1875"/>
+        <parent link="base_plate_link"/>
+        <child link="standoff_rods4_link"/>
+    </joint>
 </robot>

File: xacro/rviz_materials.xacro (robot description, xacro)
@@ -4,3 +4,6 @@
       <color rgba="0.0 0.0 1.0 1"/>
   </material>
+  <material name="White">
+      <color rgba="1 1 1 1"/>
+  </material>
 </robot>

Commit message: Xacro: added robot's top plate aka cup holder tray

File: xacro/barista_robot_model.urdf.xacro (robot description, xacro)
@@ -4,4 +4,5 @@
     <xacro:include filename="$(find barista_robot_description)/xacro/rviz_materials.xacro"/>
     <xacro:include filename="$(find barista_robot_description)/xacro/standoff_rods.xacro"/>
+    <xacro:include filename="$(find barista_robot_description)/xacro/cup_holder_tray.xacro"/>
     <!-- Properties -->
     <xacro:property name="base_plate_mass" value="0.8"/>
@@ -65,3 +66,10 @@
         <child link="standoff_rods4_link"/>
     </joint>
+    <!-- Cup Holder Tray -->
+    <xacro:cup_holder_tray name="cup_holder_tray_link" color="Blue"/>
+    <joint name="cup_holder_tray_joint" type="fixed">
+        <origin rpy="0 0 0" xyz="0 0 0.3425"/>
+        <parent link="base_plate_link"/>
+        <child link="cup_holder_tray_link"/>
+    </joint>
 </robot>

Commit message: Xacro: added robot's top plate aka cup holder tray

File: xacro/barista_robot_model.urdf.xacro (robot description, xacro)
@@ -4,4 +4,5 @@
     <xacro:include filename="$(find barista_robot_description)/xacro/rviz_materials.xacro"/>
     <xacro:include filename="$(find barista_robot_description)/xacro/standoff_rods.xacro"/>
+    <xacro:include filename="$(find barista_robot_description)/xacro/cup_holder_tray.xacro"/>
     <!-- Properties -->
     <xacro:property name="base_plate_mass" value="2.5"/>
@@ -65,3 +66,10 @@
         <child link="standoff_rods4_link"/>
     </joint>
+    <!-- Cup Holder Tray -->
+    <xacro:cup_holder_tray name="cup_holder_tray_link" color="Blue"/>
+    <joint name="cup_holder_tray_joint" type="fixed">
+        <origin rpy="0 0 0" xyz="0 0 0.3425"/>
+        <parent link="base_plate_link"/>
+        <child link="cup_holder_tray_link"/>
+    </joint>
 </robot>

Commit message: Xacro: added two wheels

File: xacro/barista_robot_model.urdf.xacro (robot description, xacro)
@@ -5,4 +5,5 @@
     <xacro:include filename="$(find barista_robot_description)/xacro/standoff_rods.xacro"/>
     <xacro:include filename="$(find barista_robot_description)/xacro/cup_holder_tray.xacro"/>
+    <xacro:include filename="$(find barista_robot_description)/xacro/drive_wheels.xacro"/>
     <!-- Properties -->
     <xacro:property name="base_plate_mass" value="0.8"/>
@@ -73,3 +74,23 @@
         <child link="cup_holder_tray_link"/>
     </joint>
+    <!-- Wheel Left and Right -->
+    <xacro:wheel name="left_wheel_link" color="Black"/>
+    <xacro:wheel name="right_wheel_link" color="Black"/>
+    <!-- Wheel Left and Right Joints-->
+    <joint name="left_wheel_joint" type="continuous">
+        <parent link="base_plate_link"/>
+        <child link="left_wheel_link"/>
+        <origin xyz="0.0 0.15 -0.053" rpy="-1.57 0 0"/>
+        <axis rpy="0 0 0" xyz="0 0 1"/>
+        <limit effort="10000" velocity="1000"/>
+        <joint_properties damping="1.0" friction="1.0"/>
+    </joint>
+    <joint name="right_wheel_joint" type="continuous">
+        <parent link="base_plate_link"/>
+        <child link="right_wheel_link"/>
+        <origin xyz="0.0 -0.15 -0.053" rpy="-1.57 0 0"/>
+        <axis rpy="0 0 0" xyz="0 0 1"/>
+        <limit effort="10000" velocity="1000"/>
+        <joint_properties damping="1.0" friction="1.0"/>
+    </joint>
 </robot>

Commit message: Xacro: added two wheels

File: xacro/barista_robot_model.urdf.xacro (robot description, xacro)
@@ -5,4 +5,5 @@
     <xacro:include filename="$(find barista_robot_description)/xacro/standoff_rods.xacro"/>
     <xacro:include filename="$(find barista_robot_description)/xacro/cup_holder_tray.xacro"/>
+    <xacro:include filename="$(find barista_robot_description)/xacro/drive_wheels.xacro"/>
     <!-- Properties -->
     <xacro:property name="base_plate_mass" value="0.8"/>
@@ -73,3 +74,23 @@
         <child link="cup_holder_tray_link"/>
     </joint>
+    <!-- Wheel Left and Right -->
+    <xacro:wheel name="left_wheel_link" color="Black"/>
+    <xacro:wheel name="right_wheel_link" color="Black"/>
+    <!-- Wheel Left and Right Joints-->
+    <joint name="left_wheel_joint" type="continuous">
+        <parent link="base_plate_link"/>
+        <child link="left_wheel_link"/>
+        <origin xyz="0.0 0.15 -0.053" rpy="-1.57 0 0"/>
+        <axis rpy="0 0 0" xyz="0 0 1"/>
+        <limit effort="10000" velocity="1000"/>
+        <joint_properties damping="1.0" friction="1.0"/>
+    </joint>
+    <joint name="right_wheel_joint" type="continuous">
+        <parent link="base_plate_link"/>
+        <child link="right_wheel_link"/>
+        <origin xyz="0.0 -0.15 -0.053" rpy="-1.57 0 0"/>
+        <axis rpy="0 0 0" xyz="0 0 1"/>
+        <limit effort="10000" velocity="1000"/>
+        <joint_properties damping="1.0" friction="1.0"/>
+    </joint>
 </robot>

File: xacro/rviz_materials.xacro (robot description, xacro)
@@ -7,3 +7,6 @@
       <color rgba="1 1 1 1"/>
   </material>
+  <material name="Black">
+      <color rgba="0 0 0 1"/>
+  </material>
 </robot>

Commit message: Xacro: added two wheels

File: xacro/barista_robot_model.urdf.xacro (robot description, xacro)
@@ -5,4 +5,5 @@
     <xacro:include filename="$(find barista_robot_description)/xacro/standoff_rods.xacro"/>
     <xacro:include filename="$(find barista_robot_description)/xacro/cup_holder_tray.xacro"/>
+    <xacro:include filename="$(find barista_robot_description)/xacro/drive_wheels.xacro"/>
     <!-- Properties -->
     <xacro:property name="base_plate_mass" value="2.5"/>
@@ -73,3 +74,23 @@
         <child link="cup_holder_tray_link"/>
     </joint>
+    <!-- Wheel Left and Right -->
+    <xacro:wheel name="left_wheel_link" color="Black"/>
+    <xacro:wheel name="right_wheel_link" color="Black"/>
+    <!-- Wheel Left and Right Joints-->
+    <joint name="left_wheel_joint" type="continuous">
+        <parent link="base_plate_link"/>
+        <child link="left_wheel_link"/>
+        <origin xyz="0.0 0.15 -0.07" rpy="-1.57 0 0"/>
+        <axis rpy="0 0 0" xyz="0 0 1"/>
+        <limit effort="10000" velocity="1000"/>
+        <joint_properties damping="1.0" friction="1.0"/>
+    </joint>
+    <joint name="right_wheel_joint" type="continuous">
+        <parent link="base_plate_link"/>
+        <child link="right_wheel_link"/>
+        <origin xyz="0.0 -0.15 -0.07" rpy="-1.57 0 0"/>
+        <axis rpy="0 0 0" xyz="0 0 1"/>
+        <limit effort="10000" velocity="1000"/>
+        <joint_properties damping="1.0" friction="1.0"/>
+    </joint>
 </robot>

File: xacro/rviz_materials.xacro (robot description, xacro)
@@ -7,3 +7,6 @@
       <color rgba="1 1 1 1"/>
   </material>
+  <material name="Black">
+      <color rgba="0 0 0 1"/>
+  </material>
 </robot>

Commit message: Xacro: added gazebo plugin for joint state publisher

File: xacro/barista_robot_model.urdf.xacro (robot description, xacro)
@@ -6,5 +6,7 @@
     <xacro:include filename="$(find barista_robot_description)/xacro/cup_holder_tray.xacro"/>
     <xacro:include filename="$(find barista_robot_description)/xacro/drive_wheels.xacro"/>
+    <xacro:include filename="$(find barista_robot_description)/xacro/gazebo_plugins.xacro"/>
     <!-- Properties -->
+    <xacro:property name="robot_name" value="barista_bot"/>
     <xacro:property name="base_plate_mass" value="0.8"/>
     <xacro:property name="base_plate_radius" value="0.178"/>
@@ -94,3 +96,10 @@
         <joint_properties damping="1.0" friction="1.0"/>
     </joint>
+    <xacro:joint_state_publisher_plugin
+        robot_name="${robot_name}"
+        rate="50"
+        joints="${[
+            'left_wheel_joint',
+            'right_wheel_joint'
+        ]}"/>
 </robot>

Commit message: Xacro: added gazebo plugin for joint state publisher

File: xacro/barista_robot_model.urdf.xacro (robot description, xacro)
@@ -6,5 +6,7 @@
     <xacro:include filename="$(find barista_robot_description)/xacro/cup_holder_tray.xacro"/>
     <xacro:include filename="$(find barista_robot_description)/xacro/drive_wheels.xacro"/>
+    <xacro:include filename="$(find barista_robot_description)/xacro/gazebo_plugins.xacro"/>
     <!-- Properties -->
+    <xacro:property name="robot_name" value="barista_bot"/>
     <xacro:property name="base_plate_mass" value="2.5"/>
     <xacro:property name="base_plate_radius" value="0.178"/>
@@ -94,3 +96,10 @@
         <joint_properties damping="1.0" friction="1.0"/>
     </joint>
+    <xacro:joint_state_publisher_plugin
+        robot_name="${robot_name}"
+        rate="50"
+        joints="${[
+            'left_wheel_joint',
+            'right_wheel_joint'
+        ]}"/>
 </robot>

Commit message: Xacro: added differential drive gazebo plugin

File: xacro/barista_robot_model.urdf.xacro (robot description, xacro)
@@ -103,3 +103,10 @@
             'right_wheel_joint'
         ]}"/>
+    <xacro:differential_drive_controller_plugin
+        robot_name="${robot_name}"
+        base_frame="base_link"
+        left_joint="left_wheel_joint"
+        right_joint="right_wheel_joint"
+        separation="0.30"
+        diameter="0.0704" />
 </robot>

File: xacro/gazebo_plugins.xacro (robot description, xacro)
@@ -29,3 +29,24 @@
             'right_wheel_joint'
         ]}"/> -->
+    <!-- Differential drive -->
+    <xacro:macro name="differential_drive_controller_plugin" params="robot_name base_frame left_joint right_joint separation diameter">
+        <gazebo>
+            <plugin filename="libgazebo_ros_diff_drive.so" name="${robot_name}_differential_drive_controller">
+            <!-- wheels -->
+            <left_joint>${left_joint}</left_joint>
+            <right_joint>${right_joint}</right_joint>
+            <!-- kinematics -->
+            <wheel_separation>${separation}</wheel_separation>
+            <wheel_diameter>${diameter}</wheel_diameter>
+            <!-- limits -->
+            <max_wheel_torque>1.0</max_wheel_torque>
+            <max_wheel_acceleration>2.0</max_wheel_acceleration>
+            <!-- output -->
+            <publish_odom>true</publish_odom>
+            <publish_odom_tf>true</publish_odom_tf>
+            <odometry_frame>odom</odometry_frame>
+            <robot_base_frame>${base_frame}</robot_base_frame>
+            </plugin>
+        </gazebo>
+    </xacro:macro>
 </robot>

Commit message: Xacro: Added caster wheels

File: xacro/barista_robot_model.urdf.xacro (robot description, xacro)
@@ -7,4 +7,5 @@
     <xacro:include filename="$(find barista_robot_description)/xacro/drive_wheels.xacro"/>
     <xacro:include filename="$(find barista_robot_description)/xacro/gazebo_plugins.xacro"/>
+    <xacro:include filename="$(find barista_robot_description)/xacro/caster_wheels.xacro"/>
     <!-- Properties -->
     <xacro:property name="robot_name" value="barista_bot"/>
@@ -96,11 +97,4 @@
         <joint_properties damping="1.0" friction="1.0"/>
     </joint>
-    <xacro:joint_state_publisher_plugin
-        robot_name="${robot_name}"
-        rate="50"
-        joints="${[
-            'left_wheel_joint',
-            'right_wheel_joint'
-        ]}"/>
     <xacro:differential_drive_controller_plugin
         robot_name="${robot_name}"
@@ -110,3 +104,32 @@
         separation="0.30"
         diameter="0.0704" />
+    <xacro:caster_wheels prefix="front"
+        pos_x="0.150"
+        pos_y="0"
+        pos_z="-0.0730"
+        parent_link="base_plate_link"
+        color_roll="Red"
+        color_pitch="Green"
+        color_yaw="Blue" />
+    <xacro:caster_wheels prefix="back"
+        pos_x="-0.150"
+        pos_y="0"
+        pos_z="-0.0730"
+        parent_link="base_plate_link"
+        color_roll="Red"
+        color_pitch="Green"
+        color_yaw="Blue" />
+    <xacro:joint_state_publisher_plugin
+        robot_name="${robot_name}"
+        rate="50"
+        joints="${[
+            'left_wheel_joint',
+            'right_wheel_joint',
+            'front_roll_joint',
+            'front_pitch_joint',
+            'front_yaw_joint',
+            'back_roll_joint',
+            'back_pitch_joint',
+            'back_yaw_joint'
+        ]}"/>
 </robot>

File: xacro/rviz_materials.xacro (robot description, xacro)
@@ -10,3 +10,9 @@
       <color rgba="0 0 0 1"/>
   </material>
+  <material name="Red">
+      <color rgba="1 0 0 1"/>
+  </material>
+  <material name="Green">
+      <color rgba="0 1 0 1"/>
+  </material>
 </robot>

Commit message: Xacro: Added Laser Scanner & its plugin

File: xacro/barista_robot_model.urdf.xacro (robot description, xacro)
@@ -8,4 +8,7 @@
     <xacro:include filename="$(find barista_robot_description)/xacro/gazebo_plugins.xacro"/>
     <xacro:include filename="$(find barista_robot_description)/xacro/caster_wheels.xacro"/>
+    <xacro:include filename="$(find barista_robot_description)/xacro/laser_scanner.xacro"/>
+    <!-- Arguments -->
+    <xacro:arg name="include_laser" default="true"/>
     <!-- Properties -->
     <xacro:property name="robot_name" value="barista_bot"/>
@@ -120,4 +123,19 @@
         color_pitch="Green"
         color_yaw="Blue" />
+    <!-- Laser Scanner -->
+    <xacro:if value="$(arg include_laser)">
+        <xacro:laser_scanner
+            name="laser_scanner"
+            color="Green"
+            ray_pos="0.0 0.0 0.047" />
+        <joint name="laser_scanner_joint" type="fixed">
+            <origin rpy="0 0 0" xyz="0.10 0.0 0.0775"/>
+            <parent link="base_plate_link"/>
+            <child link="laser_scanner_link"/>
+        </joint>
+        <xacro:laser_scanner_plugin
+            link_name="laser_scanner_ray_link"
+            out_topic="scan"/>
+    </xacro:if>
     <xacro:joint_state_publisher_plugin
         robot_name="${robot_name}"

File: xacro/gazebo_plugins.xacro (robot description, xacro)
@@ -50,3 +50,36 @@
         </gazebo>
     </xacro:macro>
+    <!-- Laser Scanner Plugin -->
+    <xacro:macro name="laser_scanner_plugin" params="link_name out_topic">
+        <gazebo reference="${link_name}">
+            <sensor name="sensor_ray" type="ray">
+                <pose>0 0 0 0 0 0</pose>
+                <ray>
+                    <scan>
+                        <horizontal>
+                            <samples>720</samples>
+                            <resolution>0.5</resolution>
+                            <min_angle>-3.1416</min_angle>
+                            <max_angle>3.1416</max_angle>
+                        </horizontal>
+                    </scan>
+                    <range>
+                        <min>0.07</min>
+                        <max>10.0</max>
+                        <resolution>0.01</resolution>
+                    </range>
+                </ray>
+                <always_on>true</always_on>
+                <visualize>true</visualize>
+                <update_rate>50.0</update_rate>
+                <plugin name="laser" filename="libgazebo_ros_ray_sensor.so">
+                    <ros>
+                        <!-- <namespace>/barista_bot</namespace> -->
+                        <remapping>~/out:=${out_topic}</remapping>
+                    </ros>
+                    <output_type>sensor_msgs/LaserScan</output_type>
+                </plugin>
+            </sensor>
+        </gazebo>
+    </xacro:macro>
 </robot>
