Commit message: Xacro: added laser scanner

File: xacro/barista_robot_model.urdf.xacro (robot description, xacro)
@@ -8,4 +8,5 @@
     <xacro:include filename="$(find barista_robot_description)/xacro/gazebo_plugins.xacro"/>
     <xacro:include filename="$(find barista_robot_description)/xacro/caster_wheels.xacro"/>
+    <xacro:include filename="$(find barista_robot_description)/xacro/laser_scanner.xacro"/>
     <!-- Properties -->
     <xacro:property name="robot_name" value="barista_bot"/>
@@ -120,4 +121,19 @@
         color_pitch="Green"
         color_yaw="Blue" />
+    <!-- Laser Scanner -->
+    <!-- Link representing the laser -->
+    <link name="laser_scanner_ray_link"/>
+    <!-- Joint connecting base_link and front_laser -->
+    <joint name="laser_scanner_ray_joint" type="fixed">
+        <origin rpy="0 0 0" xyz="0.10 0.0 0.14"/>
+        <parent link="base_plate_link" />
+        <child link="laser_scanner_ray_link" />
+    </joint>
+    <xacro:laser_scanner name="laser_scanner_link" color="Green"/>
+    <joint name="laser_scanner_joint" type="fixed">
+        <origin rpy="0 0 0" xyz="0.10 0.0 0.0775"/>
+        <parent link="base_plate_link"/>
+        <child link="laser_scanner_link"/>
+    </joint>
     <xacro:joint_state_publisher_plugin
         robot_name="${robot_name}"
@@ -133,3 +149,33 @@
             'back_yaw_joint'
         ]}"/>
+    <gazebo reference="laser_scanner_ray_link">
+        <sensor name="sensor_ray" type="ray">
+            <pose>0 0 0 0 0 0</pose>
+            <ray>
+                <scan>
+                    <horizontal>
+                        <samples>720</samples>
+                        <resolution>0.5</resolution>
+                        <min_angle>-3.1416</min_angle>
+                        <max_angle>3.1416</max_angle>
+                    </horizontal>
+                </scan>
+                <range>
+                    <min>0.07</min>
+                    <max>10.0</max>
+                    <resolution>0.01</resolution>
+                </range>
+            </ray>
+            <always_on>true</always_on>
+            <visualize>true</visualize>
+            <update_rate>35.0</update_rate>
+            <plugin name="laser" filename="libgazebo_ros_ray_sensor.so">
+                <ros>
+                    <!-- <namespace>/barista_bot</namespace> -->
+                    <remapping>~/out:=scan</remapping>
+                </ros>
+                <output_type>sensor_msgs/LaserScan</output_type>
+            </plugin>
+        </sensor>
+    </gazebo>
 </robot>

Commit message: saved tests

File: xacro/barista_robot_model.urdf.xacro (robot description, xacro)
@@ -11,6 +11,10 @@
     <!-- Arguments -->
     <xacro:arg name="include_laser" default="true"/>
+    <xacro:arg name="robot_name" default="barista"/>
+    <xacro:arg name="link_joint_prefix" default=""/>
+    <xacro:arg name="color" default="Blue"/>
     <!-- Properties -->
-    <xacro:property name="robot_name" value="barista_bot"/>
+    <xacro:property name="robot_name" value="$(arg robot_name)"/>
+    <xacro:property name="link_joint_prefix" value="$(arg link_joint_prefix)"/>
     <xacro:property name="base_plate_mass" value="0.8"/>
     <xacro:property name="base_plate_radius" value="0.178"/>
@@ -20,11 +24,11 @@
     <xacro:property name="iyy" value="${(1/12.0) * base_plate_mass * (3 * pow(base_plate_radius, 2) + pow(base_plate_length, 2))}"/>
     <xacro:property name="izz" value="${0.5 * base_plate_mass * pow(base_plate_radius, 2)}"/>
-    <link name="base_link"/>
-    <link name="base_plate_link">
+    <link name="${link_joint_prefix}base_link"/>
+    <link name="${link_joint_prefix}base_plate_link">
         <visual>
             <geometry>
                 <cylinder radius="${base_plate_radius}" length="${base_plate_length}"/>
             </geometry>
-            <material name="Blue"/>
+            <material name="$(arg color)"/>
         </visual>
         <collision>
@@ -39,52 +43,52 @@
         </inertial>
     </link>
-    <gazebo reference="base_plate_link">
-        <material>Gazebo/Blue</material>
+    <gazebo reference="${link_joint_prefix}base_plate_link">
+        <material>Gazebo/$(arg color)</material>
     </gazebo>
-    <joint name="base_link_joint" type="fixed">
+    <joint name="${link_joint_prefix}base_link_joint" type="fixed">
         <origin rpy="0 0 0" xyz="0 0 0"/>
-        <parent link="base_link"/>
-        <child link="base_plate_link"/>
+        <parent link="${link_joint_prefix}base_link"/>
+        <child link="${link_joint_prefix}base_plate_link"/>
     </joint>
     <!-- Standoff Rods -->
-    <xacro:standoff_rods name="standoff_rods1_link" color="White"/>
-    <xacro:standoff_rods name="standoff_rods2_link" color="White"/>
-    <xacro:standoff_rods name="standoff_rods3_link" color="White"/>
-    <xacro:standoff_rods name="standoff_rods4_link" color="White"/>
+    <xacro:standoff_rods name="${link_joint_prefix}standoff_rods1_link" color="White"/>
+    <xacro:standoff_rods name="${link_joint_prefix}standoff_rods2_link" color="White"/>
+    <xacro:standoff_rods name="${link_joint_prefix}standoff_rods3_link" color="White"/>
+    <xacro:standoff_rods name="${link_joint_prefix}standoff_rods4_link" color="White"/>
     <!-- Standoff Rods Joints-->
-    <joint name="standoff_rods1_joint" type="fixed">
+    <joint name="${link_joint_prefix}standoff_rods1_joint" type="fixed">
         <origin rpy="0 0 0" xyz="0.03 0.13 0.1875"/>
-        <parent link="base_plate_link"/>
-        <child link="standoff_rods1_link"/>
+        <parent link="${link_joint_prefix}base_plate_link"/>
+        <child link="${link_joint_prefix}standoff_rods1_link"/>
     </joint>
-    <joint name="standoff_rods2_joint" type="fixed">
+    <joint name="${link_joint_prefix}standoff_rods2_joint" type="fixed">
         <origin rpy="0 0 0" xyz="-0.03 0.13 0.1875"/>
-        <parent link="base_plate_link"/>
-        <child link="standoff_rods2_link"/>
+        <parent link="${link_joint_prefix}base_plate_link"/>
+        <child link="${link_joint_prefix}standoff_rods2_link"/>
     </joint>
-    <joint name="standoff_rods3_joint" type="fixed">
+    <joint name="${link_joint_prefix}standoff_rods3_joint" type="fixed">
         <origin rpy="0 0 0" xyz="-0.03 -0.13 0.1875"/>
-        <parent link="base_plate_link"/>
-        <child link="standoff_rods3_link"/>
+        <parent link="${link_joint_prefix}base_plate_link"/>
+        <child link="${link_joint_prefix}standoff_rods3_link"/>
     </joint>
-    <joint name="standoff_rods4_joint" type="fixed">
+    <joint name="${link_joint_prefix}standoff_rods4_joint" type="fixed">
         <origin rpy="0 0 0" xyz="0.03 -0.13 0.1875"/>
-        <parent link="base_plate_link"/>
-        <child link="standoff_rods4_link"/>
+        <parent link="${link_joint_prefix}base_plate_link"/>
+        <child link="${link_joint_prefix}standoff_rods4_link"/>
     </joint>
     <!-- Cup Holder Tray -->
-    <xacro:cup_holder_tray name="cup_holder_tray_link" color="Blue"/>
-    <joint name="cup_holder_tray_joint" type="fixed">
+    <xacro:cup_holder_tray name="${link_joint_prefix}cup_holder_tray_link" color="$(arg color)"/>
+    <joint name="${link_joint_prefix}cup_holder_tray_joint" type="fixed">
         <origin rpy="0 0 0" xyz="0 0 0.3425"/>
-        <parent link="base_plate_link"/>
-        <child link="cup_holder_tray_link"/>
+        <parent link="${link_joint_prefix}base_plate_link"/>
+        <child link="${link_joint_prefix}cup_holder_tray_link"/>
     </joint>
     <!-- Wheel Left and Right -->
-    <xacro:wheel name="left_wheel_link" color="Black"/>
-    <xacro:wheel name="right_wheel_link" color="Black"/>
+    <xacro:wheel name="${link_joint_prefix}left_wheel_link" color="Black"/>
+    <xacro:wheel name="${link_joint_prefix}right_wheel_link" color="Black"/>
     <!-- Wheel Left and Right Joints-->
-    <joint name="left_wheel_joint" type="continuous">
-        <parent link="base_plate_link"/>
-        <child link="left_wheel_link"/>
+    <joint name="${link_joint_prefix}left_wheel_joint" type="continuous">
+        <parent link="${link_joint_prefix}base_plate_link"/>
+        <child link="${link_joint_prefix}left_wheel_link"/>
         <origin xyz="0.0 0.15 -0.053" rpy="-1.57 0 0"/>
         <axis rpy="0 0 0" xyz="0 0 1"/>
@@ -92,7 +96,7 @@
         <joint_properties damping="1.0" friction="1.0"/>
     </joint>
-    <joint name="right_wheel_joint" type="continuous">
-        <parent link="base_plate_link"/>
-        <child link="right_wheel_link"/>
+    <joint name="${link_joint_prefix}right_wheel_joint" type="continuous">
+        <parent link="${link_joint_prefix}base_plate_link"/>
+        <child link="${link_joint_prefix}right_wheel_link"/>
         <origin xyz="0.0 -0.15 -0.053" rpy="-1.57 0 0"/>
         <axis rpy="0 0 0" xyz="0 0 1"/>
@@ -101,23 +105,23 @@
     </joint>
     <xacro:differential_drive_controller_plugin
-        robot_name="${robot_name}"
-        base_frame="base_link"
-        left_joint="left_wheel_joint"
-        right_joint="right_wheel_joint"
+        robot_name="$(arg robot_name)"
+        base_frame="${link_joint_prefix}base_link"
+        left_joint="${link_joint_prefix}left_wheel_joint"
+        right_joint="${link_joint_prefix}right_wheel_joint"
         separation="0.30"
         diameter="0.0704" />
-    <xacro:caster_wheels prefix="front"
+    <xacro:caster_wheels prefix="${link_joint_prefix}front"
         pos_x="0.150"
         pos_y="0"
         pos_z="-0.0730"
-        parent_link="base_plate_link"
+        parent_link="${link_joint_prefix}base_plate_link"
         color_roll="Red"
         color_pitch="Green"
         color_yaw="Blue" />
-    <xacro:caster_wheels prefix="back"
+    <xacro:caster_wheels prefix="${link_joint_prefix}back"
         pos_x="-0.150"
         pos_y="0"
         pos_z="-0.0730"
-        parent_link="base_plate_link"
+        parent_link="${link_joint_prefix}base_plate_link"
         color_roll="Red"
         color_pitch="Green"
@@ -126,19 +130,21 @@
     <xacro:if value="$(arg include_laser)">
         <xacro:laser_scanner
-            name="laser_scanner"
+            name="${link_joint_prefix}laser_scanner"
             color="Green"
             ray_pos="0.0 0.0 0.047" />
-        <joint name="laser_scanner_joint" type="fixed">
+        <joint name="${link_joint_prefix}laser_scanner_joint" type="fixed">
             <origin rpy="0 0 0" xyz="0.10 0.0 0.0775"/>
-            <parent link="base_plate_link"/>
-            <child link="laser_scanner_link"/>
+            <parent link="${link_joint_prefix}base_plate_link"/>
+            <child link="${link_joint_prefix}laser_scanner_link"/>
         </joint>
         <xacro:laser_scanner_plugin
-            link_name="laser_scanner_ray_link"
+            robot_name="$(arg robot_name)"
+            link_name="${link_joint_prefix}laser_scanner_ray_link"
             out_topic="scan"/>
     </xacro:if>
     <xacro:joint_state_publisher_plugin
-        robot_name="${robot_name}"
-        rate="50"
+        robot_name="$(arg robot_name)"
+        rate="10"
+        prefix="${link_joint_prefix}"
         joints="${[
             'left_wheel_joint',

File: xacro/gazebo_plugins.xacro (robot description, xacro)
@@ -1,8 +1,9 @@
 <?xml version="1.0"?>
 <robot xmlns:xacro="http://www.ros.org/wiki/xacro">
-    <xacro:macro name="joint_state_publisher_plugin" params="robot_name rate joints">
+    <xacro:macro name="joint_state_publisher_plugin" params="robot_name rate prefix joints">
         <gazebo>
-            <plugin name="${robot_name}_joint_state_publisher" filename="libgazebo_ros_joint_state_publisher.so">
+            <plugin name="joint_state_publisher" filename="libgazebo_ros_joint_state_publisher.so">
                 <ros>
+                    <namespace>/${robot_name}</namespace>
                     <remapping>~/out:=joint_states</remapping>
                 </ros>
@@ -16,5 +17,5 @@
             <!-- pop first item from list -->
             <xacro:property name="item" value="${joints.pop(0)}"/>
-            <joint_name>${item}</joint_name>
+            <joint_name>${prefix}${item}</joint_name>
             <!-- recursive call -->
             <xacro:joints_loop/>
@@ -33,4 +34,8 @@
         <gazebo>
             <plugin filename="libgazebo_ros_diff_drive.so" name="${robot_name}_differential_drive_controller">
+            <ros>
+                <namespace>/${robot_name}</namespace>
+                <remapping>/cmd_vel:=cmd_vel</remapping>
+            </ros>
             <!-- wheels -->
             <left_joint>${left_joint}</left_joint>
@@ -45,11 +50,11 @@
             <publish_odom>true</publish_odom>
             <publish_odom_tf>true</publish_odom_tf>
-            <odometry_frame>odom</odometry_frame>
-            <robot_base_frame>${base_frame}</robot_base_frame>
+            <odometry_frame>${robot_name}/odom</odometry_frame>
+            <robot_base_frame>${robot_name}/${base_frame}</robot_base_frame>
             </plugin>
         </gazebo>
     </xacro:macro>
     <!-- Laser Scanner Plugin -->
-    <xacro:macro name="laser_scanner_plugin" params="link_name out_topic">
+    <xacro:macro name="laser_scanner_plugin" params="robot_name link_name out_topic">
         <gazebo reference="${link_name}">
             <sensor name="sensor_ray" type="ray">
@@ -72,12 +77,12 @@
                 <always_on>true</always_on>
                 <visualize>true</visualize>
-                <update_rate>50.0</update_rate>
+                <update_rate>10.0</update_rate>
                 <plugin name="laser" filename="libgazebo_ros_ray_sensor.so">
                     <ros>
-                        <!-- <namespace>/barista_bot</namespace> -->
+                        <namespace>${robot_name}</namespace>
                         <remapping>~/out:=${out_topic}</remapping>
                     </ros>
                     <output_type>sensor_msgs/LaserScan</output_type>
-                    <frame_name>${link_name}</frame_name>
+                    <frame_name>${robot_name}/${link_name}</frame_name>
                 </plugin>
             </sensor>

Commit message: Use namespace for multi-robot spawn from same urdf

File: xacro/barista_robot_model.urdf.xacro (robot description, xacro)
@@ -10,7 +10,11 @@
     <xacro:include filename="$(find barista_robot_description)/xacro/laser_scanner.xacro"/>
     <!-- Arguments -->
+    <xacro:arg name="robot_name" default="barista"/>
+    <xacro:arg name="link_joint_prefix" default=""/>
+    <xacro:arg name="color" default="Blue"/>
     <xacro:arg name="include_laser" default="true"/>
     <!-- Properties -->
-    <xacro:property name="robot_name" value="barista_bot"/>
+    <xacro:property name="robot_name" value="$(arg robot_name)"/>
+    <xacro:property name="color" value="$(arg color)"/>
     <xacro:property name="base_plate_mass" value="0.8"/>
     <xacro:property name="base_plate_radius" value="0.178"/>
@@ -26,5 +30,5 @@
                 <cylinder radius="${base_plate_radius}" length="${base_plate_length}"/>
             </geometry>
-            <material name="Blue"/>
+            <material name="${color}"/>
         </visual>
         <collision>
@@ -40,5 +44,5 @@
     </link>
     <gazebo reference="base_plate_link">
-        <material>Gazebo/Blue</material>
+        <material>Gazebo/${color}</material>
     </gazebo>
     <joint name="base_link_joint" type="fixed">
@@ -74,5 +78,5 @@
     </joint>
     <!-- Cup Holder Tray -->
-    <xacro:cup_holder_tray name="cup_holder_tray_link" color="Blue"/>
+    <xacro:cup_holder_tray name="cup_holder_tray_link" color="${color}"/>
     <joint name="cup_holder_tray_joint" type="fixed">
         <origin rpy="0 0 0" xyz="0 0 0.3425"/>
@@ -135,4 +139,5 @@
         </joint>
         <xacro:laser_scanner_plugin
+            robot_name="${robot_name}"
             link_name="laser_scanner_ray_link"
             out_topic="scan"/>

File: xacro/gazebo_plugins.xacro (robot description, xacro)
@@ -3,6 +3,7 @@
     <xacro:macro name="joint_state_publisher_plugin" params="robot_name rate joints">
         <gazebo>
-            <plugin name="${robot_name}_joint_state_publisher" filename="libgazebo_ros_joint_state_publisher.so">
+            <plugin name="joint_state_publisher" filename="libgazebo_ros_joint_state_publisher.so">
                 <ros>
+                    <namespace>/${robot_name}</namespace>
                     <remapping>~/out:=joint_states</remapping>
                 </ros>
@@ -32,5 +33,8 @@
     <xacro:macro name="differential_drive_controller_plugin" params="robot_name base_frame left_joint right_joint separation diameter">
         <gazebo>
-            <plugin filename="libgazebo_ros_diff_drive.so" name="${robot_name}_differential_drive_controller">
+            <plugin filename="libgazebo_ros_diff_drive.so" name="differential_drive_controller">
+            <ros>
+                <namespace>/${robot_name}</namespace>
+            </ros>
             <!-- wheels -->
             <left_joint>${left_joint}</left_joint>
@@ -45,11 +49,11 @@
             <publish_odom>true</publish_odom>
             <publish_odom_tf>true</publish_odom_tf>
-            <odometry_frame>odom</odometry_frame>
-            <robot_base_frame>${base_frame}</robot_base_frame>
+            <odometry_frame>${robot_name}/odom</odometry_frame>
+            <robot_base_frame>${robot_name}/${base_frame}</robot_base_frame>
             </plugin>
         </gazebo>
     </xacro:macro>
     <!-- Laser Scanner Plugin -->
-    <xacro:macro name="laser_scanner_plugin" params="link_name out_topic">
+    <xacro:macro name="laser_scanner_plugin" params="robot_name link_name out_topic">
         <gazebo reference="${link_name}">
             <sensor name="sensor_ray" type="ray">
@@ -75,9 +79,9 @@
                 <plugin name="laser" filename="libgazebo_ros_ray_sensor.so">
                     <ros>
-                        <!-- <namespace>/barista_bot</namespace> -->
+                        <namespace>/${robot_name}</namespace>
                         <remapping>~/out:=${out_topic}</remapping>
                     </ros>
                     <output_type>sensor_msgs/LaserScan</output_type>
-                    <frame_name>${link_name}</frame_name>
+                    <frame_name>${robot_name}/${link_name}</frame_name>
                 </plugin>
             </sensor>
