Commit message: URDF: added four standoff rods

File: urdf/barista_robot_model.urdf (robot description, URDF)
Before this commit: robot barista_bot, 2 links, 1 joints
Links:
- added link standoff_rods1_link, mass 0.05; collision cylinder length=0.220 radius=0.010; visual cylinder length=0.220 radius=0.010
- added link standoff_rods2_link, mass 0.05; collision cylinder length=0.220 radius=0.010; visual cylinder length=0.220 radius=0.010
- added link standoff_rods3_link, mass 0.05; collision cylinder length=0.220 radius=0.010; visual cylinder length=0.220 radius=0.010
- added link standoff_rods4_link, mass 0.05; collision cylinder length=0.220 radius=0.010; visual cylinder length=0.220 radius=0.010
Joints:
- added joint standoff_rods1_joint: type fixed, parent base_plate_link, child standoff_rods1_link, origin xyz=0.03 0.13 0.1875 rpy=0 0 0
- added joint standoff_rods2_joint: type fixed, parent base_plate_link, child standoff_rods2_link, origin xyz=-0.03 0.13 0.1875 rpy=0 0 0
- added joint standoff_rods3_joint: type fixed, parent base_plate_link, child standoff_rods3_link, origin xyz=-0.03 -0.13 0.1875 rpy=0 0 0
- added joint standoff_rods4_joint: type fixed, parent base_plate_link, child standoff_rods4_link, origin xyz=0.03 -0.13 0.1875 rpy=0 0 0

Commit message: URDF: Added laser scanner link

File: urdf/barista_robot_model.urdf (robot description, URDF)
Before this commit: robot barista_bot, 6 links, 5 joints
Links:
- added link laser_scanner_link, mass 0.05; collision cylinder length=0.0275 radius=0.030; visual cylinder length=0.0275 radius=0.030
Joints:
- added joint laser_scanner_joint: type continuous, parent base_plate_link, child laser_scanner_link, origin xyz=0.10 0.0 0.09125 rpy=0 0 0

Commit message: URDF: added cup holder and joint state publisher node

File: urdf/barista_robot_model.urdf (robot description, URDF)
Before this commit: robot barista_bot, 7 links, 6 joints
Links:
- added link cup_holder_tray_link, mass 0.4; collision cylinder length=0.090 radius=0.160; visual cylinder length=0.090 radius=0.160
Joints:
- added joint cup_holder_tray_joint: type fixed, parent base_plate_link, child cup_holder_tray_link, origin xyz=0 0 0.3425 rpy=0 0 0
- joint laser_scanner_joint: axis (none) -> 0 0 1

Commit message: URDF: Added two wheels

File: urdf/barista_robot_model.urdf (robot description, URDF)
Before this commit: robot barista_bot, 8 links, 7 joints
Links:
- added link left_wheel_link, mass 2.8498940e-02; collision cylinder length=0.0206 radius=0.0352; visual cylinder length=0.0206 radius=0.0352
- added link right_wheel_link, mass 2.8498940e-02; collision cylinder length=0.0206 radius=0.0352; visual cylinder length=0.0206 radius=0.0352
Joints:
- added joint left_wheel_joint: type continuous, parent base_plate_link, child left_wheel_link, origin xyz=0.0 0.15 -0.060 rpy=-1.57 0 0, axis 0 0 1, limit effort=10000 velocity=1000
- added joint right_wheel_joint: type continuous, parent base_plate_link, child right_wheel_link, origin xyz=0.0 -0.15 -0.060 rpy=-1.57 0 0, axis 0 0 1, limit effort=10000 velocity=1000

Commit message: URDF: added caster wheels

File: urdf/barista_robot_model.urdf (robot description, URDF)
Before this commit: robot barista_bot, 10 links, 9 joints
Links:
- added link back_pitch_link; visual sphere radius=0.010
- added link back_roll_link; visual cylinder length=0.005 radius=0.010
- added link back_yaw_link; visual cylinder length=0.005 radius=0.010
- added link front_pitch_link; visual sphere radius=0.010
- added link front_roll_link; visual cylinder length=0.005 radius=0.010
- added link front_yaw_link; visual cylinder length=0.005 radius=0.010
Joints:
- added joint back_pitch_joint: type continuous, parent back_roll_link, child back_pitch_link, origin xyz=0 0 0 rpy=0 0 0, axis 0 1 0, limit effort=1000.0 velocity=100.0
- added joint back_roll_joint: type continuous, parent back_yaw_link, child back_roll_link, origin xyz=0 0 0 rpy=0 0 0, axis 1 0 0, limit effort=1000.0 velocity=100.0
- added joint back_yaw_joint: type continuous, parent base_plate_link, child back_yaw_link, origin xyz=-0.150 0 -0.075 rpy=0 0 0, axis 0 0 1, limit effort=1000.0 velocity=100.0
- added joint front_pitch_joint: type continuous, parent front_roll_link, child front_pitch_link, origin xyz=0 0 0 rpy=0 0 0, axis 0 1 0, limit effort=1000.0 velocity=100.0
- added joint front_roll_joint: type continuous, parent front_yaw_link, child front_roll_link, origin xyz=0 0 0 rpy=0 0 0, axis 1 0 0, limit effort=1000.0 velocity=100.0
- added joint front_yaw_joint: type continuous, parent base_plate_link, child front_yaw_link, origin xyz=0.150 0 -0.075 rpy=0 0 0, axis 0 0 1, limit effort=1000.0 velocity=100.0

Commit message: Adjust parameters

File: urdf/barista_robot_model.urdf (robot description, URDF)
Before this commit: robot barista_bot, 16 links, 15 joints
Links:
- link back_pitch_link: geometry visual sphere radius=0.0150
- link back_roll_link: geometry visual cylinder length=0.005 radius=0.0150
- link back_yaw_link: geometry visual cylinder length=0.005 radius=0.0150
- link front_pitch_link: geometry visual sphere radius=0.0150
- link front_roll_link: geometry visual cylinder length=0.005 radius=0.0150
- link front_yaw_link: geometry visual cylinder length=0.005 radius=0.0150
Joints:
- joint back_yaw_joint: origin xyz=-0.150 0 -0.075 rpy=0 0 0 -> xyz=-0.150 0 -0.0730 rpy=0 0 0
- joint front_yaw_joint: origin xyz=0.150 0 -0.075 rpy=0 0 0 -> xyz=0.150 0 -0.0730 rpy=0 0 0
- joint left_wheel_joint: origin xyz=0.0 0.15 -0.060 rpy=-1.57 0 0 -> xyz=0.0 0.15 -0.0528 rpy=-1.57 0 0
- joint right_wheel_joint: origin xyz=0.0 -0.15 -0.060 rpy=-1.57 0 0 -> xyz=0.0 -0.15 -0.0528 rpy=-1.57 0 0

Commit message: Added mesh file for laser scanner

File: urdf/barista_robot_model.urdf (robot description, URDF)
Before this commit: robot barista_bot, 16 links, 15 joints
Links:
- link laser_scanner_link: geometry collision cylinder length=0.0275 radius=0.030; visual mesh filename=package://barista_robot_description/meshes/hokuyo_urg_04lx.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 scale=1.0 1.0 1.0

Commit message: Added ros2 control for laser scanner

File: urdf/barista_robot_model.urdf (robot description, URDF)
Before this commit: robot barista_bot, 16 links, 15 joints
Links:
- added link laser_scan_frame
Joints:
- added joint laser_scan_frame_joint: type fixed, parent base_plate_link, child laser_scan_frame, origin xyz=0.10 0.0 0.09125 rpy=0 0 0, axis 0 0 0
- joint laser_scanner_joint: limit (none) -> effort=10.0 velocity=2.0

Commit message: URDF Modifications to revisit

File: urdf/barista_robot_model.urdf (robot description, URDF)
Before this commit: robot barista_bot, 17 links, 16 joints
Links:
- link back_pitch_link: mass None -> 0.03; geometry collision sphere radius=0.0150; visual sphere radius=0.0150
- link back_roll_link: mass None -> 0.02; geometry collision cylinder length=0.005 radius=0.0150; visual cylinder length=0.005 radius=0.0150
- link back_yaw_link: mass None -> 0.02; geometry collision cylinder length=0.005 radius=0.0150; visual cylinder length=0.005 radius=0.0150
- link base_plate_link: mass 0.5 -> 0.4
- link cup_holder_tray_link: mass 0.4 -> 0.3
- link front_pitch_link: mass None -> 0.03; geometry collision sphere radius=0.0150; visual sphere radius=0.0150
- link front_roll_link: mass None -> 0.02; geometry collision cylinder length=0.005 radius=0.0150; visual cylinder length=0.005 radius=0.0150
- link front_yaw_link: mass None -> 0.02; geometry collision cylinder length=0.005 radius=0.0150; visual cylinder length=0.005 radius=0.0150
- link laser_scanner_link: mass 0.05 -> 0.2
- link left_wheel_link: mass 2.8498940e-02 -> 0.05
- link right_wheel_link: mass 2.8498940e-02 -> 0.05
- link standoff_rods1_link: mass 0.05 -> 0.03
- link standoff_rods2_link: mass 0.05 -> 0.03
- link standoff_rods3_link: mass 0.05 -> 0.03
- link standoff_rods4_link: mass 0.05 -> 0.03

Commit message: URDF: added four standoff rods

File: urdf/barista_robot_model.urdf (robot description, URDF)
Before this commit: robot barista_bot, 2 links, 1 joints
Links:
- added link standoff_rods1_link, mass 0.1; collision cylinder length=0.22 radius=0.01; visual cylinder length=0.22 radius=0.01
- added link standoff_rods2_link, mass 0.1; collision cylinder length=0.22 radius=0.01; visual cylinder length=0.22 radius=0.01
- added link standoff_rods3_link, mass 0.1; collision cylinder length=0.22 radius=0.01; visual cylinder length=0.22 radius=0.01
- added link standoff_rods4_link, mass 0.1; collision cylinder length=0.22 radius=0.01; visual cylinder length=0.22 radius=0.01
Joints:
- added joint standoff_rods1_joint: type fixed, parent base_plate_link, child standoff_rods1_link, origin xyz=0.03 0.13 0.1875 rpy=0 0 0
- added joint standoff_rods2_joint: type fixed, parent base_plate_link, child standoff_rods2_link, origin xyz=-0.03 0.13 0.1875 rpy=0 0 0
- added joint standoff_rods3_joint: type fixed, parent base_plate_link, child standoff_rods3_link, origin xyz=-0.03 -0.13 0.1875 rpy=0 0 0
- added joint standoff_rods4_joint: type fixed, parent base_plate_link, child standoff_rods4_link, origin xyz=0.03 -0.13 0.1875 rpy=0 0 0

Commit message: URDF: Added cup holder tray

File: urdf/barista_robot_model.urdf (robot description, URDF)
Before this commit: robot barista_bot, 6 links, 5 joints
Links:
- added link cup_holder_tray_link, mass 0.05; collision cylinder length=0.09 radius=0.16; visual cylinder length=0.09 radius=0.16
Joints:
- added joint cup_holder_tray_joint: type fixed, parent base_plate_link, child cup_holder_tray_link, origin xyz=0 0 0.3425 rpy=0 0 0

Commit message: URDF: Added two wheels, differential drive plugin and joint state publisher

File: urdf/barista_robot_model.urdf (robot description, URDF)
Before this commit: robot barista_bot, 7 links, 6 joints
Links:
- added link left_wheel_link, mass 0.07; collision cylinder length=0.0206 radius=0.0352; visual cylinder length=0.0206 radius=0.0352
- added link right_wheel_link, mass 0.07; collision cylinder length=0.0206 radius=0.0352; visual cylinder length=0.0206 radius=0.0352
Joints:
- added joint left_wheel_joint: type continuous, parent base_plate_link, child left_wheel_link, origin xyz=0.0 0.15 -0.053 rpy=-1.57 0 0, axis 0 0 1, limit effort=10000 velocity=1000
- added joint right_wheel_joint: type continuous, parent base_plate_link, child right_wheel_link, origin xyz=0.0 -0.15 -0.053 rpy=-1.57 0 0, axis 0 0 1, limit effort=10000 velocity=1000

Commit message: URDF: Added caster wheels

File: urdf/barista_robot_model.urdf (robot description, URDF)
Before this commit: robot barista_bot, 9 links, 8 joints
Links:
- added link back_pitch_link, mass 0.002; collision sphere radius=0.015; visual sphere radius=0.015
- added link back_roll_link, mass 0.0015; collision cylinder length=0.005 radius=0.015; visual cylinder length=0.005 radius=0.015
- added link back_yaw_link, mass 0.0015; collision cylinder length=0.005 radius=0.015; visual cylinder length=0.005 radius=0.015
- added link front_pitch_link, mass 0.002; collision sphere radius=0.015; visual sphere radius=0.015
- added link front_roll_link, mass 0.0015; collision cylinder length=0.005 radius=0.015; visual cylinder length=0.005 radius=0.015
- added link front_yaw_link, mass 0.0015; collision cylinder length=0.005 radius=0.015; visual cylinder length=0.005 radius=0.015
Joints:
- added joint back_pitch_joint: type continuous, parent back_roll_link, child back_pitch_link, origin xyz=0 0 0 rpy=0 0 0, axis 0 1 0, limit effort=1000.0 velocity=100.0
- added joint back_roll_joint: type continuous, parent back_yaw_link, child back_roll_link, origin xyz=0 0 0 rpy=0 0 0, axis 1 0 0, limit effort=1000.0 velocity=100.0
- added joint back_yaw_joint: type continuous, parent base_plate_link, child back_yaw_link, origin xyz=-0.15 0 -0.073 rpy=0 0 0, axis 0 0 1, limit effort=1000.0 velocity=100.0
- added joint front_pitch_joint: type continuous, parent front_roll_link, child front_pitch_link, origin xyz=0 0 0 rpy=0 0 0, axis 0 1 0, limit effort=1000.0 velocity=100.0
- added joint front_roll_joint: type continuous, parent front_yaw_link, child front_roll_link, origin xyz=0 0 0 rpy=0 0 0, axis 1 0 0, limit effort=1000.0 velocity=100.0
- added joint front_yaw_joint: type continuous, parent base_plate_link, child front_yaw_link, origin xyz=0.15 0 -0.073 rpy=0 0 0, axis 0 0 1, limit effort=1000.0 velocity=100.0

Commit message: URDF: Added laser scanner, model and gazebo plugin

File: urdf/barista_robot_model.urdf (robot description, URDF)
Before this commit: robot barista_bot, 15 links, 14 joints
Links:
- added link laser_scanner_link, mass 0.01; collision cylinder length=0.040 radius=0.03; visual cylinder length=0.040 radius=0.03
- added link laser_scanner_ray_link
Joints:
- added joint laser_scanner_joint: type fixed, parent base_plate_link, child laser_scanner_link, origin xyz=0.10 0.0 0.0975 rpy=0 0 0
- added joint laser_scanner_ray_joint: type fixed, parent laser_scanner_link, child laser_scanner_ray_link, origin xyz=0.0 0.0 0.0 rpy=0 0 0

Commit message: URDF: Added Hukoyo mesh for Laser, gazebo world

File: urdf/barista_robot_model.urdf (robot description, URDF)
Before this commit: robot barista_bot, 17 links, 16 joints
Links:
- link laser_scanner_link: geometry collision cylinder length=0.040 radius=0.03; visual mesh filename=package://barista_robot_description/meshes/hokuyo_urg_04lx.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 scale=1.0 1.0 1.0
Joints:
- joint laser_scanner_joint: origin xyz=0.10 0.0 0.0975 rpy=0 0 0 -> xyz=0.10 0.0 0.0775 rpy=0 0 0
- joint laser_scanner_ray_joint: origin xyz=0.0 0.0 0.0 rpy=0 0 0 -> xyz=0.0 0.0 0.047 rpy=0 0 0
